File: hardware/attiny85/microdrummer_uno.kicad_pcb (KiCad board)
At the start: 2 copper layers, 19 x 106.5 mm, 41 parts, among them M1 LITTLEBITS_MALE, M2 LITTLEBITS_FEMALE, U1 ATmega328-MMH, U2 MIC5219-5.0YM5, Y1 20MHz

Commit message: rescued symbols and migrated to kicad symbols
Parts:
- C5: value 10μF -> 2.2μF
- D6: footprint Diode_SMD:D_SOD-323F -> Diodes_SMD:D_0603
Connections:
- Jin1 pad 1: GND -> (no net)
- Jin1 pad 2: GND -> (no net)
- Jin1 pad 3: /RAW_SIGNAL -> (no net)
- Jout1 pad 1: GND -> (no net)
- Jout1 pad 2: Net-(Jout1-Pad2) -> (no net)
- Jout1 pad 3: /OUTPUT -> (no net)
