File: hardware/attiny85/microdrummer_uno.sch (KiCad schematic (older format))
At the start: 34 parts, among them M1 LITTLEBITS_MALE, M2 LITTLEBITS_FEMALE, U1 ATmega328-MMH, U2 MIC5219-5.0YM5, Y1 20MHz

Commit message: rescued symbols and migrated to kicad symbols
Parts:
- ISP1: symbol microdrummer-rescue:AVR-ISP-6 -> Connector:AVR-ISP-6
- Jin1, Jout1: symbol Miasma_IO_smd-cache:Thonk -> Connector:AudioJack2_SwitchT
- M1: symbol SparkFun-Connectors:LITTLEBITS_MALE -> microdrummer_uno-rescue:LITTLEBITS_MALE-SparkFun-Connectors
- M2: symbol SparkFun-Connectors:LITTLEBITS_FEMALE -> microdrummer_uno-rescue:LITTLEBITS_FEMALE-SparkFun-Connectors
- Qin1, Qout1: symbol Miasma_IO_smd-cache:MMBT3904 -> Transistor_BJT:MMBT3904
- SELout1: symbol Switch1:SW_SPDT -> Switch:SW_SPDT
- bclr1, bin1, brec1: symbol Switch1:SW_SPST -> Switch:SW_SPST
Connections:
- net GND: now also Jin1.S, Jin1.TN, Jout1.S; no longer Jin1.1, Jin1.2, Jout1.1
- net OUTPUT: now also Jout1.T; no longer Jout1.3
- net RAW_SIGNAL: now also Jin1.T; no longer Jin1.3
Changed lines of the file:
@@
 $EndDescr
 $Comp
-L Switch1:SW_SPST bin1
+L Switch:SW_SPST bin1
 U 1 1 5B3956B4
 P 5400 4150
@@
 $EndComp
 $Comp
-L Switch1:SW_SPST bclr1
+L Switch:SW_SPST bclr1
 U 1 1 5B395716
 P 5400 3250
@@
 BTN_CLR
 $Comp
-L microdrummer-rescue:AVR-ISP-6 ISP1
-U 1 1 5C24387F
-P 6450 5300
-F 0 "ISP1" H 6345 5540 50  0000 C CNN
-F 1 "AVR-ISP-6" H 6185 5070 50  0000 L BNN
-F 2 "Pin_Headers:Pin_Header_Straight_2x03_Pitch2.54mm" V 5930 5340 50  0001 C CNN
-F 3 "" H 6425 5300 50  0001 C CNN
-	1    6450 5300
-	1    0    0    -1
-$EndComp
-$Comp
-L Miasma_IO_smd-cache:Thonk Jin1
+L Connector:AudioJack2_SwitchT Jin1
 U 1 1 5C52850D
-P 1250 3200
-F 0 "Jin1" H 1250 3200 60  0000 C CNN
-F 1 "Thonk" H 1250 3350 60  0000 C CNN
-F 2 "chillpizza:schurter_3.5mm_mono_audio" H 1250 3200 60  0001 C CNN
-F 3 "" H 1250 3200 60  0000 C CNN
-	1    1250 3200
+P 1350 3300
+F 0 "Jin1" H 1350 3300 60  0000 C CNN
+F 1 "Thonk" H 1350 3450 60  0000 C CNN
+F 2 "chillpizza:schurter_3.5mm_mono_audio" H 1350 3300 60  0001 C CNN
+F 3 "" H 1350 3300 60  0000 C CNN
+	1    1350 3300
 	1    0    0    -1
 $EndComp
@@
 $EndComp
 $Comp
-L Miasma_IO_smd-cache:MMBT3904 Qin1
+L Transistor_BJT:MMBT3904 Qin1
 U 1 1 5C528741
 P 2350 3300
@@
 RAW_OUTPUT
 Wire Wire Line
-	1550 3000 1550 3100
-Wire Wire Line
 	2050 2800 2050 2900
 Wire Wire Line
@@
 	5700 3250 5600 3250
 $Comp
-L SparkFun-Connectors:LITTLEBITS_FEMALE M2
+L microdrummer_uno-rescue:LITTLEBITS_FEMALE-SparkFun-Connectors M2
 U 1 1 5C670B33
 P 10750 850
@@
 $EndComp
 $Comp
-L SparkFun-Connectors:LITTLEBITS_MALE M1
+L microdrummer_uno-rescue:LITTLEBITS_MALE-SparkFun-Connectors M1
 U 1 1 5C670BF7
 P 8950 850
@@
 $EndComp
 $Comp
-L Switch1:SW_SPDT SELout1
+L Switch:SW_SPDT SELout1
 U 1 1 5C6726D5
 P 2150 4700
@@
 Text Label 1950 4600 2    60   ~ 0
 OUT_TRIGGER
-Connection ~ 1550 3100
 $Comp
 L power:GND #PWR019
@@
 	1    0    0    -1
 $EndComp
-Wire Wire Line
-	3250 6200 3250 6300
-NoConn ~ 3250 6100
-$Comp
-L Miasma_IO_smd-cache:Thonk Jout1
+NoConn ~ 3250 5900
+$Comp
+L Connector:AudioJack2_SwitchT Jout1
 U 1 1 5C53024A
-P 3550 6100
-F 0 "Jout1" H 3550 6100 60  0000 C CNN
-F 1 "Thonk" H 3550 6250 60  0000 C CNN
-F 2 "chillpizza:schurter_3.5mm_mono_audio" H 3550 6100 60  0001 C CNN
-F 3 "" H 3550 6100 60  0000 C CNN
-	1    3550 6100
+P 3450 6000
+F 0 "Jout1" H 3450 6000 60  0000 C CNN
+F 1 "Thonk" H 3450 6150 60  0000 C CNN
+F 2 "chillpizza:schurter_3.5mm_mono_audio" H 3450 6000 60  0001 C CNN
+F 3 "" H 3450 6000 60  0000 C CNN
+	1    3450 6000
 	-1   0    0    1
 $EndComp
@@
 $EndComp
 $Comp
-L Miasma_IO_smd-cache:MMBT3904 Qout1
+L Transistor_BJT:MMBT3904 Qout1
 U 1 1 5C71A36D
 P 1850 7050
@@
 Wire Wire Line
 	2050 3300 2150 3300
-Wire Wire Line
-	1550 3100 1550 3200
 Wire Wire Line
 	1650 6000 2050 6000
@@
 	2400 6000 2750 6000
 $Comp
-L Switch1:SW_SPST brec1
+L Switch:SW_SPST brec1
 U 1 1 5F1FF126
 P 5400 3700
@@
 Wire Wire Line
 	5700 3700 5600 3700
-Wire Wire Line
-	6550 5200 6900 5200
-Wire Wire Line
-	6900 5200 6900 5050
-Wire Wire Line
-	6550 5300 6900 5300
-Wire Wire Line
-	6550 5400 6900 5400
-Wire Wire Line
-	6900 5400 6900 5550
-Wire Wire Line
-	6300 5200 6000 5200
-Wire Wire Line
-	6000 5200 6000 5050
-Wire Wire Line
-	6300 5300 6000 5300
-Wire Wire Line
-	6300 5400 6000 5400
-Wire Wire Line
-	6000 5400 6000 5550
-Text Label 6900 5300 0    50   ~ 0
-ISP_MOSI
-Text Label 6000 5050 2    50   ~ 0
-ISP_MISO
-Text Label 6000 5300 2    50   ~ 0
+Text Label 7200 5300 0    50   ~ 0
 ISP_SCK
-Text Label 6000 5550 2    50   ~ 0
-ISP_RST
 $Comp
 L power:GND #PWR0113
 U 1 1 5F225406
-P 6900 5550
-F 0 "#PWR0113" H 6900 5300 50  0001 C CNN
-F 1 "GND" H 6905 5377 50  0000 C CNN
-F 2 "" H 6900 5550 50  0001 C CNN
-F 3 "" H 6900 5550 50  0001 C CNN
-	1    6900 5550
+P 6350 5850
+F 0 "#PWR0113" H 6350 5600 50  0001 C CNN
+F 1 "GND" H 6355 5677 50  0000 C CNN
+F 2 "" H 6350 5850 50  0001 C CNN
+F 3 "" H 6350 5850 50  0001 C CNN
+	1    6350 5850
 	1    0    0    -1
 $EndComp
@@
 L power:+5V #PWR0114
 U 1 1 5F225A1B
-P 6900 5050
-F 0 "#PWR0114" H 6900 4900 50  0001 C CNN
-F 1 "+5V" H 6915 5223 50  0000 C CNN
-F 2 "" H 6900 5050 50  0001 C CNN
-F 3 "" H 6900 5050 50  0001 C CNN
-	1    6900 5050
+P 6350 4650
+F 0 "#PWR0114" H 6350 4500 50  0001 C CNN
+F 1 "+5V" H 6365 4823 50  0000 C CNN
+F 2 "" H 6350 4650 50  0001 C CNN
+F 3 "" H 6350 4650 50  0001 C CNN
+	1    6350 4650
 	1    0    0    -1
 $EndComp
@@
 $EndComp
 $Comp
-L Miasma_IO_smd-cache:+12V #PWR0106
+L power:+12V #PWR0106
 U 1 1 5F24B4FF
 P 2100 1050
@@
 $EndComp
 $Comp
-L Miasma_IO_smd-cache:+12V #PWR0117
+L power:+12V #PWR0117
 U 1 1 5F24BB02
 P 1000 1050
@@
 NoConn ~ 9800 4850
 NoConn ~ 9800 4750
+Wire Wire Line
+	1550 3000 1550 3200
+$Comp
+L power:GND #PWR?
+U 1 1 601A523B
+P 1400 3750
+F 0 "#PWR?" H 1400 3500 50  0001 C CNN
+F 1 "GND" H 1405 3577 50  0000 C CNN
+F 2 "" H 1400 3750 50  0001 C CNN
+F 3 "" H 1400 3750 50  0001 C CNN
+	1    1400 3750
+	1    0    0    -1
+$EndComp
+Wire Wire Line
+	1400 3750 1400 3600
+Wire Wire Line
+	1400 3600 1550 3600
+Wire Wire Line
+	1550 3600 1550 3400
+Wire Wire Line
+	3250 6100 3250 6300
+Wire Wire Line
+	6850 5200 7200 5200
+Text Label 7200 5200 0    50   ~ 0
+ISP_MOSI
+$Comp
+L Connector:AVR-ISP-6 ISP1
+U 1 1 5C24387F
+P 6450 5300
+F 0 "ISP1" H 6345 5540 50  0000 C CNN
+F 1 "AVR-ISP-6" H 6185 5070 50  0000 L BNN
+F 2 "Pin_Headers:Pin_Header_Straight_2x03_Pitch2.54mm" V 5930 5340 50  0001 C CNN
+F 3 "" H 6425 5300 50  0001 C CNN
+	1    6450 5300
+	1    0    0    -1
+$EndComp
+Text Label 7200 5100 0    50   ~ 0
+ISP_MISO
+Wire Wire Line
+	7200 5100 6850 5100
+Wire Wire Line
+	7200 5300 6850 5300
+Text Label 7200 5400 0    50   ~ 0
+ISP_RST
+Wire Wire Line
+	7200 5400 6850 5400
+Wire Wire Line
+	6350 4650 6350 4800
+Wire Wire Line
+	6350 5700 6350 5850
 $EndSCHEMATC
