File: hardware/nologic/nologic_front.sch (KiCad schematic (older format))
At the start: 42 parts, among them J1 Conn_01x05_Male, J3 AudioJack2_SwitchT, J4 AudioJack2_SwitchT, SW1 Rotary_Encoder_Switch, SW2 SW_SPST, SW3 SW_SPST

Commit message: starting rear panel
Connections:
- net at D27.1 (DOUT): now also D26.3 (DIN); no longer D28.3 (DIN)
- net at D27.3 (DIN): now also D28.1 (DOUT); no longer D26.1 (DOUT)
- net at D11.1 (DOUT): now also D10.3 (DIN); no longer D12.3 (DIN)
- net at D11.3 (DIN): now also D12.1 (DOUT); no longer D10.1 (DOUT)
- net at D13.3 (DIN): now also D14.1 (DOUT); no longer D12.1 (DOUT)
- net at D29.3 (DIN): now also D30.1 (DOUT); no longer D28.1 (DOUT)
- net at D25.1 (DOUT): now also D33.2 (DIN); no longer D26.3 (DIN)
- net at D25.3 (DIN): now also D26.1 (DOUT); no longer D17.1 (DOUT)
- net at D9.1 (DOUT): now also D24.3 (DIN); no longer D10.3 (DIN)
- net at D9.3 (DIN): now also D10.1 (DOUT); no longer D1.1 (DOUT)
- net at D32.3 (DIN): now also D17.1 (DOUT); no longer D31.1 (DOUT)
- net at D31.3 (DIN): now also D32.1 (DOUT); no longer D30.1 (DOUT)
- net at D16.3 (DIN): now also D1.1 (DOUT); no longer D15.1 (DOUT)
- net at D15.3 (DIN): now also D16.1 (DOUT); no longer D14.1 (DOUT)
- net at D29.1 (DOUT): now also D28.3 (DIN); no longer D30.3 (DIN)
- net at D13.1 (DOUT): now also D12.3 (DIN); no longer D14.3 (DIN)
- new net: D30.3 (DIN), D31.1 (DOUT)
- new net: D14.3 (DIN), D15.1 (DOUT)
Changed lines of the file:
@@
 	1450 1300 1450 900
-Wire Wire Line
-	1450 900  3400 900
-Wire Wire Line
-	3400 900  3400 1300
-Wire Wire Line
-	2800 1300 2800 2250
-Wire Wire Line
-	3400 2250 3400 3100
-Wire Wire Line
-	2800 3100 2800 3900
-Wire Wire Line
-	3400 3900 3400 4750
-Wire Wire Line
-	2800 4750 2800 5550
-Wire Wire Line
-	3400 5550 3400 6350
-Wire Wire Line
-	3400 7200 4150 7200
 Wire Wire Line
 	4750 7200 4750 6350
@@
 Wire Wire Line
 	4150 1300 4150 900
-Wire Wire Line
-	4150 900  6100 900
-Wire Wire Line
-	6100 900  6100 1300
-Wire Wire Line
-	5500 1300 5500 2250
-Wire Wire Line
-	6100 2250 6100 3100
-Wire Wire Line
-	5500 3100 5500 3900
-Wire Wire Line
-	6100 3900 6100 4750
-Wire Wire Line
-	5500 4750 5500 5550
-Wire Wire Line
-	6100 5550 6100 6350
-Wire Wire Line
-	5500 6350 5500 7200
-Wire Wire Line
-	6100 7200 6450 7200
-Wire Wire Line
-	6450 7200 6450 2750
 $Comp
 L Connector:AudioJack2_SwitchT J4
@@
 Wire Wire Line
 	10850 5850 10650 5850
-Wire Wire Line
-	2800 6350 2800 7200
 $Comp
 L power:VDD #PWR0104
@@
 NoConn ~ 9700 1650
 NoConn ~ 9700 1750
+Wire Wire Line
+	1450 900  2450 900
+Wire Wire Line
+	2450 900  2450 7200
+Wire Wire Line
+	2450 7200 2800 7200
+Wire Wire Line
+	3400 7200 3400 6350
+Wire Wire Line
+	2800 6350 2800 5550
+Wire Wire Line
+	3400 5550 3400 4750
+Wire Wire Line
+	2800 4750 2800 3900
+Wire Wire Line
+	3400 3900 3400 3100
+Wire Wire Line
+	2800 3100 2800 2250
+Wire Wire Line
+	3400 2250 3400 1300
+Wire Wire Line
+	2800 1300 2800 900
+Wire Wire Line
+	2800 900  3800 900
+Wire Wire Line
+	3800 900  3800 7200
+Wire Wire Line
+	3800 7200 4150 7200
+Wire Wire Line
+	4150 900  5150 900
+Wire Wire Line
+	5150 900  5150 7200
+Wire Wire Line
+	5150 7200 5500 7200
+Wire Wire Line
+	6100 7200 6100 6350
+Wire Wire Line
+	5500 6350 5500 5550
+Wire Wire Line
+	6100 5550 6100 4750
+Wire Wire Line
+	5500 4750 5500 3900
+Wire Wire Line
+	6100 3900 6100 3100
+Wire Wire Line
+	5500 3100 5500 2250
+Wire Wire Line
+	6100 2250 6100 1300
+Wire Wire Line
+	5500 1300 5500 900
+Wire Wire Line
+	5500 900  6450 900
+Wire Wire Line
+	6450 900  6450 2750
 $EndSCHEMATC
