File: hardware/nologic/nologic_front.kicad_pcb (KiCad board)
At the start: 2 copper layers, 25 x 128.5 mm, 49 parts, among them J1 Conn_01x03_Female, J2 Conn_01x05_Female, J3 AudioJack2_SwitchT, J4 AudioJack2_SwitchT, J5 Conn_01x03_Female, J6 Conn_01x03_Female, J7 Conn_01x02_Female, J8 Conn_01x02_Female, SW1 Rotary_Encoder_Switch, SW2 SW_SPST, SW3 SW_SPST

Commit message: starting rear panel
Parts:
- removed the G*** at (136.8, 115.0)
- removed J2: Conn_01x05_Female, Connector_PinHeader_2.54mm:PinHeader_1x05_P2.54mm_Vertical
- removed J5, J6: Conn_01x03_Female, Connector_PinHeader_2.54mm:PinHeader_1x03_P2.54mm_Vertical
- removed J7, J8: Conn_01x02_Female, Connector_PinHeader_2.54mm:PinHeader_1x02_P2.54mm_Vertical
- D1, D10, D11, D12, D13, D14, D15, D16, D17, D18, D19, D2, D20, D21, D22, D23, D24, D25, D26, D27, D28, D29, D3, D30, D31, D32, D4, D5, D6, D7, D8, D9: footprint chillpizza:LED_SK6812MINI_PLCC4_3.5x3.5mm_P1.75mm -> chillpizza:LED_SK6812MINI_PLCC4_3.5x3.5mm_P1.75mm_flush
- J1: value Conn_01x03_Female -> Conn_01x05_Male; footprint Connector_PinHeader_2.54mm:PinHeader_1x03_P2.54mm_Vertical -> Connector_PinSocket_2.54mm:PinSocket_1x05_P2.54mm_Vertical_SMD_Pin1Left; moved to B.Cu
- J3, J4: footprint chillpizza:schurter_3.5mm_mono_audio_kicad -> chillpizza:Jack_3.5mm_QingPu_WQP-PJ3410_Vertical_Top
- SW1: footprint Keebio-Parts:RotaryEncoder_Alps_EC11E-Switch_Vertical_H20mm -> chillpizza:Rotary_Encoder_Switched_PEC11R_top
- moved J1 26.2 mm to (124.3, 136.3), turned to 270 degrees
- moved D33 7.77 mm to (129.3, 74.5), turned to 180 degrees
- moved D34 6.75 mm to (119.3, 74.5), turned to 180 degrees
- moved SW1 6.70 mm to (124.3, 131.0), turned to 90 degrees
- moved D1 1.00 mm to (117.1, 78.3), turned to 270 degrees
- moved D10 1.00 mm to (121.9, 83.1)
- moved D11 1.00 mm to (121.9, 87.9), turned to 270 degrees
- moved D12 1.00 mm to (121.9, 92.8)
- moved D13 1.00 mm to (121.9, 97.6), turned to 270 degrees
- moved D14 1.00 mm to (121.9, 102.4)
- moved D15 1.00 mm to (121.9, 107.3), turned to 270 degrees
- moved D16 1.00 mm to (121.9, 112.1)
- moved D17 1.00 mm to (126.7, 78.3), turned to 270 degrees
- moved D18 1.00 mm to (126.7, 83.1)
- moved D19 1.00 mm to (126.7, 87.9), turned to 270 degrees
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Connections:
- D1 pad 2: Net-(D1-Pad2) -> GND
- D1 pad 4: Net-(D1-Pad4) -> VDD
- D10 pad 2: Net-(D1-Pad2) -> GND
- D10 pad 4: Net-(D1-Pad4) -> VDD
- D11 pad 1: Net-(D11-Pad1) -> Net-(D10-Pad3)
- D11 pad 2: Net-(D1-Pad2) -> GND
- D11 pad 4: Net-(D1-Pad4) -> VDD
- D12 pad 1: Net-(D12-Pad1) -> Net-(D11-Pad3)
- D12 pad 2: Net-(D1-Pad2) -> GND
- D12 pad 4: Net-(D1-Pad4) -> VDD
- D13 pad 1: Net-(D13-Pad1) -> Net-(D12-Pad3)
- D13 pad 2: Net-(D1-Pad2) -> GND
- D13 pad 4: Net-(D1-Pad4) -> VDD
- D14 pad 1: Net-(D14-Pad1) -> Net-(D13-Pad3)
- D14 pad 2: Net-(D1-Pad2) -> GND
- D14 pad 4: Net-(D1-Pad4) -> VDD
- D15 pad 1: Net-(D15-Pad1) -> Net-(D14-Pad3)
- D15 pad 2: Net-(D1-Pad2) -> GND
- D15 pad 4: Net-(D1-Pad4) -> VDD
- D16 pad 1: Net-(D16-Pad1) -> Net-(D15-Pad3)
- D16 pad 2: Net-(D1-Pad2) -> GND
- D16 pad 3: Net-(D16-Pad3) -> Net-(D1-Pad1)
- D16 pad 4: Net-(D1-Pad4) -> VDD
- D17 pad 2: Net-(D1-Pad2) -> GND
- D17 pad 4: Net-(D1-Pad4) -> VDD
- D18 pad 1: Net-(D18-Pad1) -> Net-(D17-Pad3)
- D18 pad 2: Net-(D1-Pad2) -> GND
- D18 pad 3: Net-(D10-Pad1) -> Net-(D18-Pad3)
- D18 pad 4: Net-(D1-Pad4) -> VDD
- D19 pad 1: Net-(D11-Pad3) -> Net-(D18-Pad3)
- D19 pad 2: Net-(D1-Pad2) -> GND
- D19 pad 4: Net-(D1-Pad4) -> VDD
- D2 pad 1: Net-(D10-Pad3) -> Net-(D1-Pad3)
- D2 pad 2: Net-(D1-Pad2) -> GND
- D2 pad 4: Net-(D1-Pad4) -> VDD
- D20 pad 1: Net-(D20-Pad1) -> Net-(D19-Pad3)
- D20 pad 2: Net-(D1-Pad2) -> GND
- D20 pad 3: Net-(D12-Pad1) -> Net-(D20-Pad3)
- D20 pad 4: Net-(D1-Pad4) -> VDD
- D21 pad 1: Net-(D13-Pad3) -> Net-(D20-Pad3)
- D21 pad 2: Net-(D1-Pad2) -> GND
- D21 pad 4: Net-(D1-Pad4) -> VDD
- D22 pad 1: Net-(D22-Pad1) -> Net-(D21-Pad3)
- D22 pad 2: Net-(D1-Pad2) -> GND
- D22 pad 3: Net-(D14-Pad1) -> Net-(D22-Pad3)
- D22 pad 4: Net-(D1-Pad4) -> VDD
- D23 pad 1: Net-(D15-Pad3) -> Net-(D22-Pad3)
- D23 pad 2: Net-(D1-Pad2) -> GND
- D23 pad 4: Net-(D1-Pad4) -> VDD
- D24 pad 1: Net-(D24-Pad1) -> Net-(D23-Pad3)
- D24 pad 2: Net-(D1-Pad2) -> GND
- D24 pad 3: Net-(D16-Pad1) -> Net-(D24-Pad3)
- D24 pad 4: Net-(D1-Pad4) -> VDD
- D25 pad 1: Net-(D17-Pad3) -> Net-(D25-Pad1)
- D25 pad 2: Net-(D1-Pad2) -> GND
- D25 pad 4: Net-(D1-Pad4) -> VDD
- D26 pad 2: Net-(D1-Pad2) -> GND
- D26 pad 3: Net-(D18-Pad1) -> Net-(D26-Pad3)
- D26 pad 4: Net-(D1-Pad4) -> VDD
- D27 pad 1: Net-(D19-Pad3) -> Net-(D26-Pad3)
- D27 pad 2: Net-(D1-Pad2) -> GND
- D27 pad 4: Net-(D1-Pad4) -> VDD
- D28 pad 2: Net-(D1-Pad2) -> GND
- D28 pad 3: Net-(D20-Pad1) -> Net-(D28-Pad3)
- D28 pad 4: Net-(D1-Pad4) -> VDD
- D29 pad 1: Net-(D21-Pad3) -> Net-(D28-Pad3)
- D29 pad 2: Net-(D1-Pad2) -> GND
- D29 pad 4: Net-(D1-Pad4) -> VDD
- D3 pad 2: Net-(D1-Pad2) -> GND
- D3 pad 3: Net-(D11-Pad1) -> Net-(D3-Pad3)
- D3 pad 4: Net-(D1-Pad4) -> VDD
- D30 pad 2: Net-(D1-Pad2) -> GND
- D30 pad 3: Net-(D22-Pad1) -> Net-(D30-Pad3)
- D30 pad 4: Net-(D1-Pad4) -> VDD
- D31 pad 1: Net-(D23-Pad3) -> Net-(D30-Pad3)
- D31 pad 2: Net-(D1-Pad2) -> GND
- D31 pad 4: Net-(D1-Pad4) -> VDD
- D32 pad 2: Net-(D1-Pad2) -> GND
- D32 pad 3: Net-(D24-Pad1) -> Net-(D17-Pad1)
- D32 pad 4: Net-(D1-Pad4) -> VDD
- D33 pad 1: Net-(D1-Pad2) -> GND
- D33 pad 2: Net-(D1-Pad1) -> Net-(D25-Pad1)
- D33 pad 3: Net-(D1-Pad4) -> VDD
- D34 pad 1: Net-(D1-Pad2) -> GND
- D34 pad 3: Net-(D1-Pad4) -> VDD
- D4 pad 1: Net-(D12-Pad3) -> Net-(D3-Pad3)
- D4 pad 2: Net-(D1-Pad2) -> GND
- D4 pad 4: Net-(D1-Pad4) -> VDD
- D5 pad 2: Net-(D1-Pad2) -> GND
- D5 pad 3: Net-(D13-Pad1) -> Net-(D5-Pad3)
- D5 pad 4: Net-(D1-Pad4) -> VDD
- D6 pad 1: Net-(D14-Pad3) -> Net-(D5-Pad3)
- D6 pad 2: Net-(D1-Pad2) -> GND
- D6 pad 4: Net-(D1-Pad4) -> VDD
- D7 pad 2: Net-(D1-Pad2) -> GND
- D7 pad 3: Net-(D15-Pad1) -> Net-(D7-Pad3)
- D7 pad 4: Net-(D1-Pad4) -> VDD
- D8 pad 1: Net-(D16-Pad3) -> Net-(D7-Pad3)
- D8 pad 2: Net-(D1-Pad2) -> GND
- D8 pad 4: Net-(D1-Pad4) -> VDD
- D9 pad 1: Net-(D1-Pad3) -> Net-(D24-Pad3)
- D9 pad 2: Net-(D1-Pad2) -> GND
- D9 pad 3: Net-(D17-Pad1) -> Net-(D10-Pad1)
- D9 pad 4: Net-(D1-Pad4) -> VDD
- J1 pad 1: Net-(D1-Pad2) -> VDD
- J1 pad 2: Net-(D8-Pad3) -> Net-(J1-Pad2)
- J1 pad 3: Net-(D1-Pad4) -> Net-(J1-Pad3)
- SW2 pad 1: Net-(J7-Pad1) -> GND
- SW2 pad 2: Net-(J7-Pad2) -> Net-(J1-Pad3)
- SW3 pad 1: Net-(J8-Pad1) -> GND
- SW3 pad 2: Net-(J8-Pad2) -> Net-(J1-Pad2)
Routing:
- net GND: track 0.00 -> 425.8 mm, vias 0 -> 4
- net VDD: track 0.00 -> 295.2 mm, vias 0 -> 1
- net Net-(D1-Pad4): track 173.8 -> 0.00 mm, vias 1 -> 0
- net Net-(D1-Pad2): track 166.7 -> 0.00 mm, vias 1 -> 0
- net Net-(J2-Pad3): track 48.2 -> 0.00 mm
- net Net-(J8-Pad2): track 43.2 -> 0.00 mm
- net Net-(D24-Pad3): track 0.00 -> 38.6 mm
- net Net-(J4-PadS): track 35.9 -> 0.00 mm
- net Net-(D17-Pad1): track 5.17 -> 38.6 mm
- net Net-(J1-Pad3): track 0.00 -> 33.0 mm
- net Net-(J2-Pad2): track 21.5 -> 0.00 mm
- net Net-(J2-Pad1): track 20.0 -> 0.00 mm
- net Net-(J3-PadTN): track 19.0 -> 0.00 mm
- net Net-(J4-PadT): track 19.0 -> 0.00 mm
- net Net-(J4-PadTN): track 18.9 -> 0.00 mm
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Other:
- board size 25 x 128.5 mm -> 20 x 128.5 mm

Commit message: front and rear graphics
Parts:
- removed G***: LOGO, chillpizza:graphic beat farm arcs
- H1, H2: value MountingHole -> mounting_hole
- SW1: value Rotary_Encoder_Switch -> rotary_encoder_switch
Other:
- board text added: "beat farm"
- board text added: "undo redo"
