File: hardware/nologic/nologic_rear.kicad_pcb (KiCad board)
At the start: 2 copper layers, 20 x 78.2 mm, 5 parts, among them J1 Conn_01x11_Female, J2 Conn_01x05_Female, J3 AudioJack2_SwitchT, J4 AudioJack2_SwitchT, SW1 Rotary_Encoder_Switch

Commit message: front and rear graphics
Parts:
- SW1: footprint digikey-footprints:Rotary_Encoder_Switched_PEC11R -> chillpizza:Rotary_Encoder_Switched_PEC11R
Routing:
- net Net-(J1-Pad7): track 0.00 -> 30.0 mm
- net GND: track 119.6 -> 135.8 mm
- net Net-(J1-Pad9): track 34.2 -> 36.0 mm
- net Net-(J1-Pad8): track 41.7 -> 40.0 mm
- net VDD: track 28.0 -> 28.8 mm
Other:
- board text added: "5v"
- board text added: "A"
- board text added: "B"
- board text added: "C"
- board text added: "data"
- board text added: "gnd"
- board text added: "in"
- board text added: "out"
- board text added: "rec_sw"
- board text added: "rotary_sw"
- board text added: "trig_sw"
Changed lines of the file:
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@@
   (general
     (thickness 1.6)
-    (drawings 4)
-    (tracks 43)
+    (drawings 15)
+    (tracks 56)
     (zones 0)
     (modules 5)
@@
     (pad_to_mask_clearance 0.051)
     (solder_mask_min_width 0.25)
-    (aux_axis_origin 0 0)
+    (aux_axis_origin 114.3 50.8)
+    (grid_origin 114.3 50.8)
     (visible_elements FFFFFF7F)
     (pcbplotparams
@@
     )
   )
-  (module digikey-footprints:Rotary_Encoder_Switched_PEC11R (layer F.Cu)
+  (module chillpizza:Rotary_Encoder_Switched_PEC11R (layer F.Cu)
     (at 124.3 131 90)
     (fp_text reference SW1 (at 5.275 -9.4 90) (layer F.SilkS)
@@
     (pad 3 thru_hole rect (at 0 0 90) (size 2.8 3.6) (drill oval 1.8 2.6) (layers *.Cu *.Mask))
     (pad 3 thru_hole rect (at 11.4 0 90) (size 2.8 3.6) (drill oval 1.8 2.6) (layers *.Cu *.Mask))
-    (pad 1 thru_hole circle (at 3.2 -7 90) (size 2 2) (drill 1) (layers *.Cu *.Mask))
-    (pad 2 thru_hole circle (at 8.2 -7 90) (size 2 2) (drill 1) (layers *.Cu *.Mask))
+    (pad S1 thru_hole circle (at 3.2 -7 90) (size 2 2) (drill 1) (layers *.Cu *.Mask)
+      (net 7 "Net-(J1-Pad7)"))
+    (pad S2 thru_hole circle (at 8.2 -7 90) (size 2 2) (drill 1) (layers *.Cu *.Mask)
+      (net 10 GND))
     (pad A thru_hole circle (at 3.2 7.5 90) (size 2 2) (drill 1) (layers *.Cu *.Mask)
       (net 6 "Net-(J1-Pad6)"))
@@
     (pad B thru_hole circle (at 8.2 7.5 90) (size 2 2) (drill 1) (layers *.Cu *.Mask)
       (net 4 "Net-(J1-Pad4)"))
+  )
+  (gr_text rec_sw (at 127 104.775) (layer B.SilkS)
+    (effects (font (size 1 1) (thickness 0.15)) (justify right mirror))
+  )
+  (gr_text trig_sw (at 127 102.235) (layer B.SilkS)
+    (effects (font (size 1 1) (thickness 0.15)) (justify right mirror))
+  )
+  (gr_text 5v (at 127 109.855) (layer B.SilkS)
+    (effects (font (size 1 1) (thickness 0.15)) (justify right mirror))
+  )
+  (gr_text gnd (at 127 107.315) (layer B.SilkS)
+    (effects (font (size 1 1) (thickness 0.15)) (justify right mirror))
+  )
+  (gr_text rotary_sw (at 127 99.695) (layer B.SilkS)
+    (effects (font (size 1 1) (thickness 0.15)) (justify right mirror))
+  )
+  (gr_text A (at 127 97.155) (layer B.SilkS)
+    (effects (font (size 1 1) (thickness 0.15)) (justify right mirror))
+  )
+  (gr_text C (at 127 94.615) (layer B.SilkS)
+    (effects (font (size 1 1) (thickness 0.15)) (justify right mirror))
+  )
+  (gr_text B (at 127 92.075) (layer B.SilkS)
+    (effects (font (size 1 1) (thickness 0.15)) (justify right mirror))
+  )
+  (gr_text data (at 127 89.535) (layer B.SilkS)
+    (effects (font (size 1 1) (thickness 0.15)) (justify right mirror))
+  )
+  (gr_text "out\n" (at 127 86.995) (layer B.SilkS)
+    (effects (font (size 1 1) (thickness 0.15)) (justify right mirror))
+  )
+  (gr_text in (at 127 84.455) (layer B.SilkS)
+    (effects (font (size 1 1) (thickness 0.15)) (justify right mirror))
   )
   (gr_line (start 114.3 140) (end 114.3 61.8) (layer Edge.Cuts) (width 0.05))
@@
   (segment (start 129.79999 111.19999) (end 129.79999 125.371992) (width 0.4) (layer F.Cu) (net 6))
   (segment (start 115.7 97.1) (end 129.79999 111.19999) (width 0.4) (layer F.Cu) (net 6))
-  (segment (start 125.309999 135.450001) (end 124.46 136.3) (width 0.4) (layer F.Cu) (net 8))
-  (segment (start 129.199981 131.560019) (end 125.309999 135.450001) (width 0.4) (layer F.Cu) (net 8))
-  (segment (start 129.199981 115.679981) (end 129.199981 131.560019) (width 0.4) (layer F.Cu) (net 8))
-  (segment (start 115.7 102.18) (end 129.199981 115.679981) (width 0.4) (layer F.Cu) (net 8))
-  (segment (start 121.92 110.94) (end 121.92 136.3) (width 0.4) (layer F.Cu) (net 9))
-  (segment (start 115.7 104.72) (end 121.92 110.94) (width 0.4) (layer F.Cu) (net 9))
+  (segment (start 118.299999 126.800001) (end 117.3 127.8) (width 0.4) (layer F.Cu) (net 7))
+  (segment (start 118.700001 126.399999) (end 118.299999 126.800001) (width 0.4) (layer F.Cu) (net 7))
+  (segment (start 118.700001 102.640001) (end 118.700001 126.399999) (width 0.4) (layer F.Cu) (net 7))
+  (segment (start 115.7 99.64) (end 118.700001 102.640001) (width 0.4) (layer F.Cu) (net 7))
+  (segment (start 115.7 102.18) (end 117.550011 104.030011) (width 0.4) (layer F.Cu) (net 8))
+  (segment (start 117.550011 104.030011) (end 117.55001 115.698532) (width 0.4) (layer F.Cu) (net 8))
+  (segment (start 117.55001 115.698532) (end 115.32502 117.923522) (width 0.4) (layer F.Cu) (net 8))
+  (segment (start 123.610001 135.450001) (end 124.46 136.3) (width 0.4) (layer F.Cu) (net 8))
+  (segment (start 122.877999 135.450001) (end 123.610001 135.450001) (width 0.4) (layer F.Cu) (net 8))
+  (segment (start 115.32502 127.897022) (end 122.877999 135.450001) (width 0.4) (layer F.Cu) (net 8))
+  (segment (start 115.32502 117.923522) (end 115.32502 127.897022) (width 0.4) (layer F.Cu) (net 8))
+  (segment (start 116.950001 115.449999) (end 114.72501 117.67499) (width 0.4) (layer F.Cu) (net 9))
+  (segment (start 116.950001 105.970001) (end 116.950001 115.449999) (width 0.4) (layer F.Cu) (net 9))
+  (segment (start 115.7 104.72) (end 116.950001 105.970001) (width 0.4) (layer F.Cu) (net 9))
+  (segment (start 114.72501 129.10501) (end 121.92 136.3) (width 0.4) (layer F.Cu) (net 9))
+  (segment (start 114.72501 117.67499) (end 114.72501 129.10501) (width 0.4) (layer F.Cu) (net 9))
   (segment (start 115.6 70.45) (end 115.6 67.8) (width 0.4) (layer B.Cu) (net 10))
   (segment (start 116.950001 71.800001) (end 115.6 70.45) (width 0.4) (layer B.Cu) (net 10))
@@
   (segment (start 116.902081 107.26) (end 129.54 119.897919) (width 0.4) (layer B.Cu) (net 10))
   (segment (start 115.7 107.26) (end 116.902081 107.26) (width 0.4) (layer B.Cu) (net 10))
-  (segment (start 119.38 113.48) (end 119.38 136.3) (width 0.4) (layer F.Cu) (net 11))
-  (segment (start 115.7 109.8) (end 119.38 113.48) (width 0.4) (layer F.Cu) (net 11))
+  (segment (start 117.3 108.86) (end 117.3 122.8) (width 0.4) (layer B.Cu) (net 10))
+  (segment (start 115.7 107.26) (end 117.3 108.86) (width 0.4) (layer B.Cu) (net 10))
+  (segment (start 118.13 136.3) (end 119.38 136.3) (width 0.4) (layer B.Cu) (net 11))
+  (segment (start 115.7 133.87) (end 118.13 136.3) (width 0.4) (layer B.Cu) (net 11))
+  (segment (start 115.7 109.8) (end 115.7 133.87) (width 0.4) (layer B.Cu) (net 11))
 )
