File: hardware/nologic/nologic_rear.sch (KiCad schematic (older format))
At the start: 5 parts, among them J1 Conn_01x11_Female, J2 Conn_01x05_Female, J3 AudioJack2_SwitchT, J4 AudioJack2_SwitchT, SW1 Rotary_Encoder_Switch

Commit message: front and rear graphics
Parts:
- SW1: footprint digikey-footprints:Rotary_Encoder_Switched_PEC11R -> chillpizza:Rotary_Encoder_Switched_PEC11R
Changed lines of the file:
@@
 F 0 "SW1" H 5650 4267 50  0000 C CNN
 F 1 "Rotary_Encoder_Switch" H 5650 4176 50  0000 C CNN
-F 2 "digikey-footprints:Rotary_Encoder_Switched_PEC11R" H 5500 4060 50  0001 C CNN
+F 2 "chillpizza:Rotary_Encoder_Switched_PEC11R" H 5500 4060 50  0001 C CNN
 F 3 "~" H 5650 4160 50  0001 C CNN
 	1    5650 3900
